File: alimentacao/alimentaçao3.brd (EAGLE design)
At the start: 100 x 80 mm, 6 parts

Commit message: git add
Parts:
- removed +ESQUERDO: TCRT5000, TCRT5000:OPTO_TCRT5000
- removed 10KΩ, 270Ω1: (no value), rcl_robotica:0204/7
- removed 270Ω: 10KΩ, rcl_robotica:0204/7
- removed X1, X2: (no value), con-molex:KK-156-4
- added ARDUINO, ARDUINO2, ARDUINO3, CHAVE: (no value), con-molex:KK-156-2
- added BUCK: CP8-ADJ, userlib:CP8-ADJ
- added C1: 100uF, rcl_robotica:E5-4
- added C2: 10uF, rcl_robotica:E5-4
- added D1: 1N4148DO35-10, diode:DO35-10
- added PONTE_H, SERVO: (no value), con-molex:KK-156-3
- added REGULADOR: 7805TV, linear:TO220V
- added U$1: XT60, XT60 (1):XT60
Connections:
- removed net ANALOG_+ESQ.: +ESQUERDO.COLL, 10KΩ.1
- new net +12V: BUCK.IN+, CHAVE.1, D1.A, PONTE_H.3
- new net +5V: ARDUINO.2, ARDUINO2.2, ARDUINO3.2, C2.+, REGULADOR.3
- new net +6V: BUCK.OUT+, SERVO.3
- new net N$2: C1.+, D1.C, REGULADOR.1
- net GND: now also ARDUINO.1, ARDUINO2.1, ARDUINO3.1, BUCK.IN-, BUCK.OUT-, C1.-, C2.-, PONTE_H.1, PONTE_H.2, REGULADOR.2, SERVO.1, SERVO.2, U$1.-; no longer +ESQUERDO.E
- net N$1: now also CHAVE.2, U$1.+; no longer +ESQUERDO.A, 270Ω.2
Routing:
- net GND: track 0.00 -> 213.0 mm
- net +12V: track 0.00 -> 100.7 mm
- net +5V: track 0.00 -> 47.1 mm
- net N$2: track 0.00 -> 14.5 mm
- net +6V: track 0.00 -> 13.9 mm
- net N$1: track 0.00 -> 12.4 mm
Other:
- board size 100 x 80 mm -> 68.2 x 55.9 mm
